File: hardware/led-board.sch (EAGLE design)
At the start: 21 parts, among them U1 ATTINY84-20SSU

Commit message: Finished layout and silkscreen work
Parts:
- added TP_GND: (no value), microbuilder:TESTPOINT1.5X2.0MM_NOCREAM
Connections:
- net GND: now also TP_GND.P$1
Other:
- note added: "3"
- note removed: "2"
Changed lines of the file:
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@@
 <part name="C2" library="microbuilder" deviceset="CAP_CERAMIC" device="0805" value="1uF"/>
 <part name="D1" library="SparkFun-DiscreteSemi" deviceset="B340A" device="" value="BA340A"/>
+<part name="TP_GND" library="microbuilder" deviceset="TESTPOINT" device="1.5X2.0MM_NOCREAM"/>
+<part name="GND4" library="supply1" deviceset="GND" device=""/>
 </parts>
 <sheets>
@@
 swapped because of
 DO/DI swap on MCU</text>
-<text x="157.48" y="-40.64" size="5.08" layer="97">2</text>
+<text x="157.48" y="-40.64" size="5.08" layer="97">3</text>
 <text x="66.548" y="-21.844" size="2.54" layer="97">Hue Chandelier LED Board
 Copyright (c) Robert Kaye 2015</text>
@@
 <instance part="C2" gate="G$1" x="35.56" y="-17.78"/>
 <instance part="D1" gate="G$1" x="25.4" y="-17.78" rot="R270"/>
+<instance part="TP_GND" gate="G$1" x="-48.26" y="-10.16"/>
+<instance part="GND4" gate="1" x="-48.26" y="-15.24"/>
 </instances>
 <busses>
@@
 <junction x="25.4" y="-22.86"/>
 </segment>
+<segment>
+<pinref part="TP_GND" gate="G$1" pin="P$1"/>
+<pinref part="GND4" gate="1" pin="GND"/>
+<wire x1="-48.26" y1="-10.16" x2="-48.26" y2="-12.7" width="0.1524" layer="91"/>
+</segment>
 </net>
